Commit message: end version for KMU

File: rsc/aliengo/aliengo.urdf (robot description, URDF)
Before this commit: robot aliengo_description, 19 links, 18 joints
Joints:
- joint FL_calf_joint: limit (none) -> lower=-5.0 upper=-0.1 effort=45 velocity=2.5
- joint FL_hip_joint: limit (none) -> lower=-0.5 upper=0.5 effort=35 velocity=2.5
- joint FL_thigh_joint: limit (none) -> lower=-1.0 upper=4.0 effort=35 velocity=2.5
- joint FR_calf_joint: limit (none) -> lower=-5.0 upper=-0.1 effort=45 velocity=2.5
- joint FR_hip_joint: limit (none) -> lower=-0.5 upper=0.5 effort=35 velocity=2.5
- joint FR_thigh_joint: limit (none) -> lower=-1.0 upper=4.0 effort=35 velocity=2.5
- joint RL_calf_joint: limit (none) -> lower=-5.0 upper=-0.1 effort=45 velocity=2.5
- joint RL_hip_joint: limit (none) -> lower=-0.5 upper=0.5 effort=35 velocity=2.5
- joint RL_thigh_joint: limit (none) -> lower=-1.0 upper=4.0 effort=35 velocity=2.5
- joint RR_calf_joint: limit (none) -> lower=-5.0 upper=-0.1 effort=45 velocity=2.5
- joint RR_hip_joint: limit (none) -> lower=-0.5 upper=0.5 effort=35 velocity=2.5
- joint RR_thigh_joint: limit (none) -> lower=-1.0 upper=4.0 effort=35 velocity=2.5

Commit message: spasite

File: rsc/aliengo/aliengo.urdf (robot description, URDF)
Before this commit: robot aliengo_description, 19 links, 18 joints
Joints:
- joint FL_calf_joint: limit lower=-5.0 upper=-0.1 effort=45 velocity=2.5 -> lower=-5.0 upper=-0.1 effort=55 velocity=10.0
- joint FL_hip_joint: limit lower=-0.5 upper=0.5 effort=35 velocity=2.5 -> lower=-0.2 upper=0.2 effort=55 velocity=10.0
- joint FL_thigh_joint: limit lower=-1.0 upper=4.0 effort=35 velocity=2.5 -> lower=-1.0 upper=4.0 effort=55 velocity=10.0
- joint FR_calf_joint: limit lower=-5.0 upper=-0.1 effort=45 velocity=2.5 -> lower=-5.0 upper=-0.1 effort=55 velocity=10.0
- joint FR_hip_joint: limit lower=-0.5 upper=0.5 effort=35 velocity=2.5 -> lower=-0.2 upper=0.2 effort=55 velocity=10.0
- joint FR_thigh_joint: limit lower=-1.0 upper=4.0 effort=35 velocity=2.5 -> lower=-1.0 upper=4.0 effort=55 velocity=10.0
- joint RL_calf_joint: limit lower=-5.0 upper=-0.1 effort=45 velocity=2.5 -> lower=-5.0 upper=-0.1 effort=55 velocity=10.0
- joint RL_hip_joint: limit lower=-0.5 upper=0.5 effort=35 velocity=2.5 -> lower=-0.2 upper=0.2 effort=55 velocity=10.0
- joint RL_thigh_joint: limit lower=-1.0 upper=4.0 effort=35 velocity=2.5 -> lower=-1.0 upper=4.0 effort=55 velocity=10.0
- joint RR_calf_joint: limit lower=-5.0 upper=-0.1 effort=45 velocity=2.5 -> lower=-5.0 upper=-0.1 effort=55 velocity=10.0
- joint RR_hip_joint: limit lower=-0.5 upper=0.5 effort=35 velocity=2.5 -> lower=-0.2 upper=0.2 effort=55 velocity=10.0
- joint RR_thigh_joint: limit lower=-1.0 upper=4.0 effort=35 velocity=2.5 -> lower=-1.0 upper=4.0 effort=55 velocity=10.0
