Commit message: results

File: rsc/a1/urdf/a1_stair.urdf (robot description, URDF)
Before this commit: robot aliengo_description, 19 links, 18 joints
Links:
- link FL_calf: mass 0.207 -> 0.166; geometry collision box size=0.2 0.016 0.016; visual mesh filename=../meshes/calf.stl scale=1 1 1
- link FL_foot: geometry collision sphere radius=0.02; visual sphere radius=0.01
- link FL_hip: mass 1.993 -> 0.696; geometry collision cylinder length=0.04 radius=0.046; visual mesh filename=../meshes/hip.stl scale=1 1 1
- link FL_thigh: mass 0.639 -> 1.013; geometry collision box size=0.2 0.0245 0.034; visual mesh filename=../meshes/thigh.stl scale=1 1 1
- link FR_calf: mass 0.207 -> 0.166; geometry collision box size=0.2 0.016 0.016; visual mesh filename=../meshes/calf.stl scale=1 1 1
- link FR_foot: geometry collision sphere radius=0.02; visual sphere radius=0.01
- link FR_hip: mass 1.993 -> 0.696; geometry collision cylinder length=0.04 radius=0.046; visual mesh filename=../meshes/hip.stl scale=1 1 1
- link FR_thigh: mass 0.639 -> 1.013; geometry collision box size=0.2 0.0245 0.034; visual mesh filename=../meshes/thigh_mirror.stl scale=1 1 1
- link RL_calf: mass 0.207 -> 0.166; geometry collision box size=0.2 0.016 0.016; visual mesh filename=../meshes/calf.stl scale=1 1 1
- link RL_foot: geometry collision sphere radius=0.02; visual sphere radius=0.01
- link RL_hip: mass 1.993 -> 0.696; geometry collision cylinder length=0.04 radius=0.046; visual mesh filename=../meshes/hip.stl scale=1 1 1
- link RL_thigh: mass 0.639 -> 1.013; geometry collision box size=0.2 0.0245 0.034; visual mesh filename=../meshes/thigh.stl scale=1 1 1
- link RR_calf: mass 0.207 -> 0.166; geometry collision box size=0.2 0.016 0.016; visual mesh filename=../meshes/calf.stl scale=1 1 1
- link RR_foot: geometry collision sphere radius=0.02; visual sphere radius=0.01
- link RR_hip: mass 1.993 -> 0.696; geometry collision cylinder length=0.04 radius=0.046; visual mesh filename=../meshes/hip.stl scale=1 1 1
- link RR_thigh: mass 0.639 -> 1.013; geometry collision box size=0.2 0.0245 0.034; visual mesh filename=../meshes/thigh_mirror.stl scale=1 1 1
- link trunk: mass 9.041 -> 4.713; geometry collision box size=0.267 0.194 0.114; visual mesh filename=../meshes/trunk.stl scale=1 1 1
Joints:
- joint FL_calf_joint: limit lower=-3.0 upper=-0.8 effort=40 velocity=15.0 -> lower=-2.6 upper=-0.9 effort=55 velocity=20.0; origin xyz=0 0 -0.25 rpy=0 0 0 -> xyz=0 0 -0.2 rpy=0 0 0
- joint FL_foot_fixed: origin xyz=0 0 -0.25 rpy=0 0 0 -> xyz=0 0 -0.2 rpy=0 0 0
- joint FL_hip_joint: limit lower=-0.25 upper=0.25 effort=40 velocity=15.0 -> lower=-0.15 upper=0.25 effort=20 velocity=50.0; origin xyz=0.2399 0.051 0 rpy=0 0 0 -> xyz=0.183 0.047 0 rpy=0 0 0
- joint FL_thigh_joint: limit lower=-1.5 upper=0.4 effort=40 velocity=15.0 -> lower=-1.0 upper=2.5 effort=55 velocity=20.0; origin xyz=0 0.083 0 rpy=0 0 0 -> xyz=0 0.08505 0 rpy=0 0 0
- joint FR_calf_joint: limit lower=-3.0 upper=-0.8 effort=40 velocity=15.0 -> lower=-2.6 upper=-0.9 effort=55 velocity=20.0; origin xyz=0 0 -0.25 rpy=0 0 0 -> xyz=0 0 -0.2 rpy=0 0 0
- joint FR_foot_fixed: origin xyz=0 0 -0.25 rpy=0 0 0 -> xyz=0 0 -0.2 rpy=0 0 0
- joint FR_hip_joint: limit lower=-0.25 upper=0.25 effort=40 velocity=15.0 -> lower=-0.25 upper=0.15 effort=20 velocity=50.0; origin xyz=0.2399 -0.051 0 rpy=0 0 0 -> xyz=0.183 -0.047 0 rpy=0 0 0
- joint FR_thigh_joint: limit lower=-1.5 upper=0.4 effort=40 velocity=15.0 -> lower=-1.0 upper=2.5 effort=55 velocity=20.0; origin xyz=0 -0.083 0 rpy=0 0 0 -> xyz=0 -0.08505 0 rpy=0 0 0
- joint RL_calf_joint: limit lower=-3.0 upper=-0.5 effort=55 velocity=15.0 -> lower=-2.6 upper=-0.95 effort=55 velocity=20.0; origin xyz=0 0 -0.25 rpy=0 0 0 -> xyz=0 0 -0.2 rpy=0 0 0
- joint RL_foot_fixed: origin xyz=0 0 -0.25 rpy=0 0 0 -> xyz=0 0 -0.2 rpy=0 0 0
- joint RL_hip_joint: limit lower=-0.25 upper=0.25 effort=55 velocity=15.0 -> lower=-0.15 upper=0.25 effort=20 velocity=50.0; origin xyz=-0.2399 0.051 0 rpy=0 0 0 -> xyz=-0.183 0.047 0 rpy=0 0 0
- joint RL_thigh_joint: limit lower=0.3 upper=0.8 effort=55 velocity=15.0 -> lower=-0.3 upper=1.9 effort=55 velocity=20.0; origin xyz=0 0.083 0 rpy=0 0 0 -> xyz=0 0.08505 0 rpy=0 0 0
- joint RR_calf_joint: limit lower=-3.0 upper=-0.5 effort=55 velocity=15.0 -> lower=-2.6 upper=-0.95 effort=55 velocity=20.0; origin xyz=0 0 -0.25 rpy=0 0 0 -> xyz=0 0 -0.2 rpy=0 0 0
- joint RR_foot_fixed: origin xyz=0 0 -0.25 rpy=0 0 0 -> xyz=0 0 -0.2 rpy=0 0 0
- joint RR_hip_joint: limit lower=-0.25 upper=0.25 effort=55 velocity=15.0 -> lower=-0.25 upper=0.15 effort=20 velocity=50.0; origin xyz=-0.2399 -0.051 0 rpy=0 0 0 -> xyz=-0.183 -0.047 0 rpy=0 0 0
- joint RR_thigh_joint: limit lower=0.3 upper=0.8 effort=55 velocity=15.0 -> lower=-0.3 upper=1.9 effort=55 velocity=20.0; origin xyz=0 -0.083 0 rpy=0 0 0 -> xyz=0 -0.08505 0 rpy=0 0 0

File: rsc/aliengo/aliengo (another copy).urdf (robot description, URDF)
Before this commit: robot aliengo_description, 19 links, 18 joints
Joints:
- joint FL_calf_joint: limit lower=-3.0 upper=-0.8 effort=40 velocity=15.0 -> lower=-4.0 upper=-0.7 effort=40 velocity=8.0
- joint FL_hip_joint: limit lower=-0.25 upper=0.25 effort=40 velocity=15.0 -> lower=-0.2 upper=0.2 effort=40 velocity=8.0
- joint FL_thigh_joint: limit lower=-1.5 upper=0.4 effort=40 velocity=15.0 -> lower=-1.5 upper=4.0 effort=40 velocity=8.0
- joint FR_calf_joint: limit lower=-3.0 upper=-0.8 effort=40 velocity=15.0 -> lower=-4.0 upper=-0.7 effort=40 velocity=8.0
- joint FR_hip_joint: limit lower=-0.25 upper=0.25 effort=40 velocity=15.0 -> lower=-0.2 upper=0.2 effort=40 velocity=8.0
- joint FR_thigh_joint: limit lower=-1.5 upper=0.4 effort=40 velocity=15.0 -> lower=-1.5 upper=4.0 effort=40 velocity=8.0
- joint RL_calf_joint: limit lower=-3.0 upper=-0.5 effort=55 velocity=15.0 -> lower=-4.0 upper=-0.1 effort=55 velocity=8.0
- joint RL_hip_joint: limit lower=-0.25 upper=0.25 effort=55 velocity=15.0 -> lower=-0.2 upper=0.2 effort=55 velocity=8.0
- joint RL_thigh_joint: limit lower=0.3 upper=0.8 effort=55 velocity=15.0 -> lower=-1.5 upper=4.0 effort=55 velocity=8.0
- joint RR_calf_joint: limit lower=-3.0 upper=-0.5 effort=55 velocity=15.0 -> lower=-4.0 upper=-0.1 effort=55 velocity=8.0
- joint RR_hip_joint: limit lower=-0.25 upper=0.25 effort=55 velocity=15.0 -> lower=-0.2 upper=0.2 effort=55 velocity=8.0
- joint RR_thigh_joint: limit lower=0.3 upper=0.8 effort=55 velocity=15.0 -> lower=-1.5 upper=4.0 effort=55 velocity=8.0
